Commit message: Changes after teleop code added

File: src/hydrogen/model/robot.xacro (robot description, xacro)
@@ -5,5 +5,6 @@
   <link name="hydrogen_frame">
     <inertial>
-      <origin xyz="0.0 0.0 -0.25" rpy="0 0 0"/>      <mass value="50.8"/>
+      <origin xyz="0.0 0.0 -0.25" rpy="0 0 0"/>
+      <mass value="40.0"/>
       <inertia ixx="0.2276" ixy="-0.004544" ixz="-0.0004496" iyy="0.1921" iyz="-0.0001196" izz="0.3559"/>
     </inertial>
@@ -59,6 +60,6 @@
                         ixx="0.00043333" iyy="0.00043333" izz="0.0008"/>
   <xacro:propeller_link name="right_propeller_1"
-                        mesh="propeller.stl"
-                        scale="0.001 0.001 0.001"
+                        mesh="propellervertical.stl"
+                        scale="0.0001 0.0001 0.0001"
                         mass="0.1"
                         ixx="0.00043333" iyy="0.00043333" izz="0.0008"/>
@@ -69,6 +70,6 @@
                         ixx="0.00043333" iyy="0.00043333" izz="0.0008"/>
   <xacro:propeller_link name="left_propeller_1"
-                        mesh="propeller.stl"
-                        scale="0.001 0.001 0.001"
+                        mesh="propellervertical.stl"
+                        scale="0.0001 0.0001 0.0001"
                         mass="0.1"
                         ixx="0.00043333" iyy="0.00043333" izz="0.0008"/>
@@ -86,5 +87,5 @@
     <parent link="hydrogen_frame"/>
     <child link="front_propeller"/>
-    <origin xyz="-0.24 -0.00725 0" rpy="0 0 0"/>
+    <origin xyz="-0.223 -0.00725 0.002" rpy="0 0 0"/>
     <axis xyz="0 0 1"/>
   </joint>
@@ -92,11 +93,11 @@
     <parent link="hydrogen_frame"/>
     <child link="left_propeller_1"/>
-    <origin xyz="-0.0527 -0.1734 0.016" rpy="0 0 0"/>
-    <axis xyz="0 1 0"/>
+    <origin xyz="-0.0631 -0.1734 0.016" rpy="-1.57 0 1.57"/>
+    <axis xyz="0 0 1"/>
   </joint>
   <joint name="left_propeller_2_joint" type="continuous">
     <parent link="hydrogen_frame"/>
     <child link="left_propeller_2"/>
-    <origin xyz="0.0527 -0.1734 0" rpy="0 0 0"/>
+    <origin xyz="0.0697 -0.1734 0.002" rpy="0 0 0"/>
     <axis xyz="0 0 1"/>
   </joint>
@@ -104,11 +105,11 @@
     <parent link="hydrogen_frame"/>
     <child link="right_propeller_1"/>
-    <origin xyz="-0.0527 0.1734 0.016" rpy="0 0 0"/>
-    <axis xyz="0 1 0"/>
+    <origin xyz="-0.0631 0.1734 0.016" rpy="-1.57 0 1.57"/>
+    <axis xyz="0 0 1"/>
   </joint>
   <joint name="right_propeller_2_joint" type="continuous">
     <parent link="hydrogen_frame"/>
     <child link="right_propeller_2"/>
-    <origin xyz="0.0527 0.1734 0" rpy="0 0 0"/>
+    <origin xyz="0.0697 0.1734 0.002" rpy="0 0 0"/>
     <axis xyz="0 0 1"/>
   </joint>
@@ -138,5 +139,4 @@
       <origin xyz="${xyz}" rpy="${rpy}"/>
     </joint>
-<!--
     <gazebo reference="${name}">
       <sensor name="${name}_depth_sensor" type="depth">
@@ -161,5 +161,4 @@
     </gazebo>
   </xacro:macro>
--->
   <xacro:zed_camera name="zed_camera_front_link" xyz="0.162 0 0.016" rpy="0 0 0"/>
   <xacro:zed_camera name="zed_camera_down_link" xyz="0.05 0 -0.08" rpy="0 1.5708 0"/>

Commit message: 9DOF IMU sensor added

File: src/hydrogen/model/robot.xacro (robot description, xacro)
@@ -5,6 +5,5 @@
   <link name="hydrogen_frame">
     <inertial>
-      <origin xyz="0.0 0.0 -0.25" rpy="0 0 0"/>
-      <mass value="40.0"/>
+      <origin xyz="0.0 0.0 -0.25" rpy="0 0 0"/>      <mass value="40.0"/>
       <inertia ixx="0.2276" ixy="-0.004544" ixz="-0.0004496" iyy="0.1921" iyz="-0.0001196" izz="0.3559"/>
     </inertial>
@@ -24,12 +23,22 @@
     </collision>
   </link>
-  <gazebo reference="hydrogen_frame">
+  <gazebo reference="base_link">
     <sensor name="imu_sensor" type="imu">
       <always_on>1</always_on>
-      <update_rate>50</update_rate>
+      <update_rate>10</update_rate>
       <visualize>true</visualize>
       <topic>imu</topic>
     </sensor>
   </gazebo>
+  <!--
+  <gazebo reference="hydrogen_frame">
+    <sensor name="magnetometer_sensor" type="magnetometer">
+      <always_on>1</always_on>
+      <update_rate>10</update_rate>
+      <visualize>true</visualize>
+      <topic>magnet</topic>
+    </sensor>
+  </gazebo>
+  -->
   <xacro:macro name="propeller_link" params="name mesh scale mass ixx iyy izz">
     <link name="${name}">

Commit message: Formatting edits made

File: src/hydrogen/model/robot.xacro (robot description, xacro)
@@ -1,14 +1,23 @@
 <?xml version="1.0"?>
 <robot xmlns:xacro="http://www.ros.org/wiki/xacro" name="Hydrogen">
-  <xacro:include filename="robot.gazebo" />
+  <xacro:include filename="robot.gazebo"/>
   <link name="base_link"/>
   <link name="hydrogen_frame">
     <inertial>
-      <origin xyz="0.0 0.0 -0.25" rpy="0 0 0"/>      <mass value="40.0"/>
-      <inertia ixx="0.2276" ixy="-0.004544" ixz="-0.0004496" iyy="0.1921" iyz="-0.0001196" izz="0.3559"/>
+      <origin xyz="0.0 0.0 -0.25" rpy="0 0 0"/>
+      <mass value="40.0"/>
+      <inertia
+        ixx="0.2276"
+        ixy="-0.004544"
+        ixz="-0.0004496"
+        iyy="0.1921"
+        iyz="-0.0001196"
+        izz="0.3559"/>
     </inertial>
     <visual>
       <geometry>
-        <mesh filename="package://hydrogen/meshes/auv2.stl" scale="0.001 0.001 0.001"/>
+        <mesh
+          filename="package://hydrogen/meshes/auv2.stl"
+          scale="0.001 0.001 0.001"/>
       </geometry>
       <material name="grey">
@@ -19,5 +28,5 @@
       <origin xyz="0.008 0.0 0.0" rpy="0 0 0"/>
       <geometry>
-       <box size="0.45 0.45 0.25"/>
+        <box size="0.45 0.45 0.25"/>
       </geometry>
     </collision>
@@ -26,5 +35,5 @@
     <sensor name="imu_sensor" type="imu">
       <always_on>1</always_on>
-      <update_rate>10</update_rate>
+      <update_rate>200</update_rate>
       <visualize>true</visualize>
       <topic>imu</topic>
@@ -33,11 +42,11 @@
   <!--
   <gazebo reference="base_link">
-  <plugin
-    filename="libauv_absolute_depth.so"
-    name="auv_absolute_depth">
-    <reference_z>0.0</reference_z>
-    <topic>/altimeter</topic>
-  </plugin>
-</gazebo>
+    <plugin
+      filename="libauv_absolute_depth.so"
+      name="auv_absolute_depth">
+      <reference_z>0.0</reference_z>
+      <topic>/altimeter</topic>
+    </plugin>
+  </gazebo>
   -->
   <xacro:macro name="propeller_link" params="name mesh scale mass ixx iyy izz">
@@ -46,9 +55,17 @@
         <origin xyz="0 0 0" rpy="0 0 0"/>
         <mass value="${mass}"/>
-        <inertia ixx="${ixx}" ixy="0" ixz="0" iyy="${iyy}" iyz="0" izz="${izz}"/>
+        <inertia
+          ixx="${ixx}"
+          ixy="0"
+          ixz="0"
+          iyy="${iyy}"
+          iyz="0"
+          izz="${izz}"/>
       </inertial>
       <visual>
         <geometry>
-          <mesh filename="package://hydrogen/meshes/${mesh}" scale="${scale}"/>
+          <mesh
+            filename="package://hydrogen/meshes/${mesh}"
+            scale="${scale}"/>
         </geometry>
         <material name="black">
@@ -58,34 +75,51 @@
       <collision>
         <geometry>
-          <mesh filename="package://hydrogen/meshes/${mesh}" scale="${scale}"/>
+          <mesh
+            filename="package://hydrogen/meshes/${mesh}"
+            scale="${scale}"/>
         </geometry>
       </collision>
     </link>
   </xacro:macro>
-  <xacro:propeller_link name="front_propeller"
-                        mesh="propellervertical.stl"
-                        scale="0.0001 0.0001 0.0001"
-                        mass="0.1"
-                        ixx="0.00043333" iyy="0.00043333" izz="0.0008"/>
-  <xacro:propeller_link name="right_propeller_1"
-                        mesh="propellervertical.stl"
-                        scale="0.0001 0.0001 0.0001"
-                        mass="0.1"
-                        ixx="0.00043333" iyy="0.00043333" izz="0.0008"/>
-  <xacro:propeller_link name="right_propeller_2"
-                        mesh="propellervertical.stl"
-                        scale="0.0001 0.0001 0.0001"
-                        mass="0.1"
-                        ixx="0.00043333" iyy="0.00043333" izz="0.0008"/>
-  <xacro:propeller_link name="left_propeller_1"
-                        mesh="propellervertical.stl"
-                        scale="0.0001 0.0001 0.0001"
-                        mass="0.1"
-                        ixx="0.00043333" iyy="0.00043333" izz="0.0008"/>
-  <xacro:propeller_link name="left_propeller_2"
-                        mesh="propellervertical.stl"
-                        scale="0.0001 0.0001 0.0001"
-                        mass="0.1"
-                        ixx="0.00043333" iyy="0.00043333" izz="0.0008"/>
+  <xacro:propeller_link
+    name="front_propeller"
+    mesh="propellervertical.stl"
+    scale="0.0001 0.0001 0.0001"
+    mass="0.1"
+    ixx="0.00043333"
+    iyy="0.00043333"
+    izz="0.0008"/>
+  <xacro:propeller_link
+    name="right_propeller_1"
+    mesh="propellervertical.stl"
+    scale="0.0001 0.0001 0.0001"
+    mass="0.1"
+    ixx="0.00043333"
+    iyy="0.00043333"
+    izz="0.0008"/>
+  <xacro:propeller_link
+    name="right_propeller_2"
+    mesh="propellervertical.stl"
+    scale="0.0001 0.0001 0.0001"
+    mass="0.1"
+    ixx="0.00043333"
+    iyy="0.00043333"
+    izz="0.0008"/>
+  <xacro:propeller_link
+    name="left_propeller_1"
+    mesh="propellervertical.stl"
+    scale="0.0001 0.0001 0.0001"
+    mass="0.1"
+    ixx="0.00043333"
+    iyy="0.00043333"
+    izz="0.0008"/>
+  <xacro:propeller_link
+    name="left_propeller_2"
+    mesh="propellervertical.stl"
+    scale="0.0001 0.0001 0.0001"
+    mass="0.1"
+    ixx="0.00043333"
+    iyy="0.00043333"
+    izz="0.0008"/>
   <joint name="base_link_joint" type="fixed">
     <parent link="base_link"/>
@@ -140,5 +174,11 @@
       <inertial>
         <mass value="0.05"/>
-        <inertia ixx="0.0001" ixy="0" ixz="0" iyy="0.0001" iyz="0" izz="0.0001"/>
+        <inertia
+          ixx="0.0001"
+          ixy="0"
+          ixz="0"
+          iyy="0.0001"
+          iyz="0"
+          izz="0.0001"/>
       </inertial>
     </link>
@@ -170,5 +210,11 @@
     </gazebo>
   </xacro:macro>
-  <xacro:zed_camera name="zed_camera_front_link" xyz="0.162 0 0.016" rpy="0 0 0"/>
-  <xacro:zed_camera name="zed_camera_down_link" xyz="0.05 0 -0.08" rpy="0 1.5708 0"/>
+  <xacro:zed_camera
+    name="zed_camera_front_link"
+    xyz="0.162 0 0.016"
+    rpy="0 0 0"/>
+  <xacro:zed_camera
+    name="zed_camera_down_link"
+    xyz="0.05 0 -0.08"
+    rpy="0 1.5708 0"/>
 </robot>

Commit message: xacro files made modular

File: src/hydrogen/model/robot.xacro (robot description, xacro)
@@ -2,233 +2,17 @@
 <robot xmlns:xacro="http://www.ros.org/wiki/xacro" name="Hydrogen">
   <xacro:include filename="robot.gazebo"/>
-  <link name="base_link"/>
-  <link name="hydrogen_frame">
-    <inertial>
-      <origin xyz="0.0 0.0 -0.25" rpy="0 0 0"/>
-      <mass value="40.0"/>
-      <inertia
-        ixx="0.2276"
-        ixy="-0.004544"
-        ixz="-0.0004496"
-        iyy="0.1921"
-        iyz="-0.0001196"
-        izz="0.3559"/>
-    </inertial>
-    <visual>
-      <geometry>
-        <mesh
-          filename="package://hydrogen/meshes/auv2.stl"
-          scale="0.001 0.001 0.001"/>
-      </geometry>
-      <material name="grey">
-        <color rgba="0.4 0.4 0.4 1"/>
-      </material>
-    </visual>
-    <collision name="hydrogen_frame_collision">
-      <origin xyz="0.008 0.0 0.0" rpy="0 0 0"/>
-      <geometry>
-        <box size="0.45 0.45 0.25"/>
-      </geometry>
-    </collision>
-  </link>
-  <gazebo reference="base_link">
-    <sensor name="imu_sensor" type="imu">
-      <always_on>1</always_on>
-      <update_rate>200</update_rate>
-      <visualize>true</visualize>
-      <topic>imu</topic>
-    </sensor>
-  </gazebo>
-  <!--
-  <gazebo reference="base_link">
-    <plugin
-      filename="libauv_absolute_depth.so"
-      name="auv_absolute_depth">
-      <reference_z>0.0</reference_z>
-      <topic>/altimeter</topic>
-    </plugin>
-  </gazebo>
-  -->
-  <xacro:macro name="propeller_link" params="name mesh scale mass ixx iyy izz">
-    <link name="${name}">
-      <inertial>
-        <origin xyz="0 0 0" rpy="0 0 0"/>
-        <mass value="${mass}"/>
-        <inertia
-          ixx="${ixx}"
-          ixy="0"
-          ixz="0"
-          iyy="${iyy}"
-          iyz="0"
-          izz="${izz}"/>
-      </inertial>
-      <visual>
-        <geometry>
-          <mesh
-            filename="package://hydrogen/meshes/${mesh}"
-            scale="${scale}"/>
-        </geometry>
-        <material name="black">
-          <color rgba="0.1 0.1 0.1 1"/>
-        </material>
-      </visual>
-      <collision>
-        <geometry>
-          <mesh
-            filename="package://hydrogen/meshes/${mesh}"
-            scale="${scale}"/>
-        </geometry>
-      </collision>
-    </link>
-  </xacro:macro>
-  <xacro:propeller_link
-    name="front_propeller"
-    mesh="propellervertical.stl"
-    scale="0.0001 0.0001 0.0001"
-    mass="0.1"
-    ixx="0.00043333"
-    iyy="0.00043333"
-    izz="0.0008"/>
-  <xacro:propeller_link
-    name="right_propeller_1"
-    mesh="propellervertical.stl"
-    scale="0.0001 0.0001 0.0001"
-    mass="0.1"
-    ixx="0.00043333"
-    iyy="0.00043333"
-    izz="0.0008"/>
-  <xacro:propeller_link
-    name="right_propeller_2"
-    mesh="propellervertical.stl"
-    scale="0.0001 0.0001 0.0001"
-    mass="0.1"
-    ixx="0.00043333"
-    iyy="0.00043333"
-    izz="0.0008"/>
-  <xacro:propeller_link
-    name="left_propeller_1"
-    mesh="propellervertical.stl"
-    scale="0.0001 0.0001 0.0001"
-    mass="0.1"
-    ixx="0.00043333"
-    iyy="0.00043333"
-    izz="0.0008"/>
-  <xacro:propeller_link
-    name="left_propeller_2"
-    mesh="propellervertical.stl"
-    scale="0.0001 0.0001 0.0001"
-    mass="0.1"
-    ixx="0.00043333"
-    iyy="0.00043333"
-    izz="0.0008"/>
-  <joint name="base_link_joint" type="fixed">
-    <parent link="base_link"/>
-    <child link="hydrogen_frame"/>
-    <origin xyz="0 0 0" rpy="0 0 0"/>
-  </joint>
-  <joint name="front_propeller_joint" type="continuous">
-    <parent link="hydrogen_frame"/>
-    <child link="front_propeller"/>
-    <origin xyz="-0.223 -0.00725 0.002" rpy="0 0 0"/>
-    <axis xyz="0 0 1"/>
-  </joint>
-  <joint name="left_propeller_1_joint" type="continuous">
-    <parent link="hydrogen_frame"/>
-    <child link="left_propeller_1"/>
-    <origin xyz="-0.0631 -0.1734 0.016" rpy="-1.57 0 1.57"/>
-    <axis xyz="0 0 1"/>
-  </joint>
-  <joint name="left_propeller_2_joint" type="continuous">
-    <parent link="hydrogen_frame"/>
-    <child link="left_propeller_2"/>
-    <origin xyz="0.0697 -0.1734 0.002" rpy="0 0 0"/>
-    <axis xyz="0 0 1"/>
-  </joint>
-  <joint name="right_propeller_1_joint" type="continuous">
-    <parent link="hydrogen_frame"/>
-    <child link="right_propeller_1"/>
-    <origin xyz="-0.0631 0.1734 0.016" rpy="-1.57 0 1.57"/>
-    <axis xyz="0 0 1"/>
-  </joint>
-  <joint name="right_propeller_2_joint" type="continuous">
-    <parent link="hydrogen_frame"/>
-    <child link="right_propeller_2"/>
-    <origin xyz="0.0697 0.1734 0.002" rpy="0 0 0"/>
-    <axis xyz="0 0 1"/>
-  </joint>
-  <xacro:macro name="zed_camera" params="name xyz rpy">
-    <link name="${name}">
-      <visual>
-        <geometry>
-          <mesh filename="package://hydrogen/meshes/zed2i.stl"/>
-        </geometry>
-        <material name="zed_mat">
-          <color rgba="0.2 0.2 0.2 1"/>
-        </material>
-      </visual>
-      <collision>
-        <geometry>
-          <mesh filename="package://hydrogen/meshes/zed2i.stl"/>
-        </geometry>
-      </collision>
-      <inertial>
-        <mass value="0.05"/>
-        <inertia
-          ixx="0.0001"
-          ixy="0"
-          ixz="0"
-          iyy="0.0001"
-          iyz="0"
-          izz="0.0001"/>
-      </inertial>
-    </link>
-    <joint name="${name}_joint" type="fixed">
-      <parent link="hydrogen_frame"/>
-      <child link="${name}"/>
-      <origin xyz="${xyz}" rpy="${rpy}"/>
-    </joint>
-    <gazebo reference="${name}">
-      <sensor name="${name}_sensor" type="rgbd_camera">
-        <always_on>true</always_on>
-        <update_rate>30</update_rate>
-        <visualize>true</visualize>
-        <!-- IMPORTANT: must match URDF link -->
-        <ignition_frame_id>${name}</ignition_frame_id>
-        <topic>${name}</topic>
-        <camera>
-          <!-- ZED 2i ~110 deg HFOV -->
-          <horizontal_fov>1.92</horizontal_fov>
-          <image>
-            <width>1280</width>
-            <height>720</height>
-            <format>R8G8B8</format>
-          </image>
-          <clip>
-            <near>0.2</near>
-            <far>20.0</far>
-          </clip>
-          <!-- Optional: reduce perfect sharpness -->
-          <noise>
-            <type>gaussian</type>
-            <mean>0.0</mean>
-            <stddev>0.002</stddev>
-          </noise>
-        </camera>
-        <!-- Depth configuration -->
-        <depth_camera>
-          <clip>
-            <near>0.2</near>
-            <far>20.0</far>
-          </clip>
-        </depth_camera>
-      </sensor>
-    </gazebo>
-  </xacro:macro>
+  <xacro:include filename="main_frame.xacro"/>
+  <xacro:hydrogen_frame/>
+  <xacro:include filename="propellers.xacro"/>
+  <xacro:propellers/>
+  <xacro:include filename="cameras.xacro"/>
   <xacro:zed_camera
     name="zed_camera_front_link"
+    parent="hydrogen_frame"
     xyz="0.162 0 0.016"
     rpy="0 0 0"/>
   <xacro:zed_camera
     name="zed_camera_down_link"
+    parent="hydrogen_frame"
     xyz="0.05 0 -0.08"
     rpy="0 1.5708 0"/>
